File: eagle/alarmClock.brd (EAGLE design)
At the start: 68.6 x 53.3 mm, 23 parts, among them T1 2SC1306, T2 2SC1306, T3 2SC1306

Commit message: Update Rev- for sending to fab
Parts:
- added R10: 147, eagle-ltspice:0204/7
- R1, R2, R3, R4, R5: value (none) -> 10k
- R6, R7, R8: value (none) -> 1k
- R9: value (none) -> 47
Connections:
- new net N$12: DAC.6, R10.1
- net N$29: now also R10.2; no longer DAC.6
Routing:
- net N$29: track 50.6 -> 22.0 mm, vias 1 -> 0
- net N$12: track 0.00 -> 18.6 mm, vias 0 -> 1
Other:
- board text added: "C:/Users/test/Documents/Arduino/Sketches/alarmClock/forkaya.bmp"
- board text added: "C:/Users/test/Documents/Arduino/Sketches/alarmClock/heart-320.bmp"
- board text removed: "For Kaya"
